Commit message: first pushing mppi version, fixed point robot urdf to have correct x and y axes

File: assets/urdf/pointRobot.urdf (robot description, URDF)
Before this commit: robot omni_base, 3 links, 2 joints
Joints:
- removed joint cart_to_pole
- added joint plane_to_link_y: type prismatic, parent link_x, child link_y, origin xyz=0 0 0, axis 0 1 0, limit effort=1000.0 velocity=100
- joint plane_to_link_x: axis 0 1 0 -> 1 0 0
