Commit message: updated urdf

File: assets/urdf/heijn.urdf (robot description, URDF)
Before this commit: robot heijn, 8 links, 7 joints
Links:
- link base_link: mass 100.0 -> 40.0
- link platform_link: mass 100.0 -> 1.0
- link pole_link: mass 100.0 -> 1.0

Commit message: First working pushing with Heijn

File: assets/urdf/heijn.urdf (robot description, URDF)
Before this commit: robot heijn, 8 links, 7 joints
Joints:
- joint mobile_joint_theta: limit lower=-5 upper=5 effort=87 velocity=2.1750 -> lower=-5 upper=5 effort=300 velocity=2.1750
- joint mobile_joint_x: limit lower=-5 upper=5 effort=87 velocity=2.1750 -> lower=-5 upper=5 effort=300 velocity=2.1750
- joint mobile_joint_y: limit lower=-5 upper=5 effort=87 velocity=2.1750 -> lower=-5 upper=5 effort=300 velocity=2.1750

Commit message: Better crate mass and shape, increased rotation limits urdf, tested pushing

File: assets/urdf/heijn.urdf (robot description, URDF)
Before this commit: robot heijn, 8 links, 7 joints
Joints:
- joint mobile_joint_theta: limit lower=-5 upper=5 effort=300 velocity=2.1750 -> lower=-5000 upper=5000 effort=300 velocity=2.1750

Commit message: make lighter and remove limits for now

File: assets/urdf/heijn.urdf (robot description, URDF)
Before this commit: robot heijn, 8 links, 7 joints
Links:
- link base_link: mass 40.0 -> 1.0
Joints:
- joint mobile_joint_theta: limit lower=-5000 upper=5000 effort=300 velocity=2.1750 -> (none)
- joint mobile_joint_x: limit lower=-5 upper=5 effort=300 velocity=2.1750 -> (none)
- joint mobile_joint_y: limit lower=-5 upper=5 effort=300 velocity=2.1750 -> (none)
