Commit message: Set rotacasters as fixed joints in urdf and set their friction to zero in isaac sim

File: assets/urdf/boxer/boxer.urdf (robot description, URDF)
Before this commit: robot albert, 8 links, 7 joints
Joints:
- joint rotacastor_left_joint: type continuous -> fixed
- joint rotacastor_right_joint: type continuous -> fixed
