Commit message: updated urdf with friction, looks like a better behavior

File: assets/urdf/objects/banana/banana.urdf (robot description, URDF)
Before this commit: robot banana, 1 links, 0 joints
Links:
- link banana: geometry collision mesh filename=objects/banana/collision.obj scale=0.01 0.01 0.01; visual mesh filename=objects/banana/textured.obj scale=0.01 0.01 0.01
