Commit message: adding hageslag, re-naming, cleanup

File: assets/urdf/omni_panda/omniPanda.urdf (robot description, URDF)
Before this commit: robot omniPanda, 13 links, 12 joints
Joints:
- joint omni_joint_theta: limit lower=-5 upper=5 effort=87 velocity=2.1750 -> lower=-500 upper=500 effort=87 velocity=2.1750
- joint omni_joint_x: limit lower=-5 upper=5 effort=87 velocity=2.1750 -> lower=-500 upper=500 effort=87 velocity=2.1750
- joint omni_joint_y: limit lower=-5 upper=5 effort=87 velocity=2.1750 -> lower=-500 upper=500 effort=87 velocity=2.1750

File: assets/urdf/omni_panda/omniPandaWithGripper.urdf (robot description, URDF)
Before this commit: robot omniPanda, 16 links, 15 joints
Joints:
- joint omni_joint_theta: limit lower=-5 upper=5 effort=87 velocity=2.1750 -> lower=-500 upper=500 effort=87 velocity=2.1750
- joint omni_joint_x: limit lower=-5 upper=5 effort=87 velocity=2.1750 -> lower=-500 upper=500 effort=87 velocity=2.1750
- joint omni_joint_y: limit lower=-5 upper=5 effort=87 velocity=2.1750 -> lower=-500 upper=500 effort=87 velocity=2.1750
