Commit message: removed limits in urdf for now

File: assets/urdf/omni_panda/omniPandaWithGripper.urdf (robot description, URDF)
Before this commit: robot omniPanda, 16 links, 15 joints
Joints:
- joint omni_joint_theta: limit lower=-500 upper=500 effort=87 velocity=2.1750 -> lower=-500 upper=500 effort=1000 velocity=500
- joint omni_joint_x: limit lower=-500 upper=500 effort=87 velocity=2.1750 -> lower=-500 upper=500 effort=1000 velocity=500
- joint omni_joint_y: limit lower=-500 upper=500 effort=87 velocity=2.1750 -> lower=-500 upper=500 effort=1000 velocity=500
