Commit message: added more accurate urdf, tested pushing hageslag size

File: assets/urdf/franka_description/robots/franka_panda_stick.urdf (robot description, URDF)
Before this commit: robot panda, 9 links, 8 joints
Links:
- added link panda_ee_tip
- link panda_ee_finger: geometry collision cylinder length=0.32 radius=0.01; visual cylinder length=0.32 radius=0.01
Joints:
- added joint panda_ee_tip: type fixed, parent panda_ee_finger, child panda_ee_tip, origin xyz=0 0 0.32 rpy=0 0 0, axis 0 0 0
