Commit message: chilled down the panda and lucky shots grabbing bananas

File: assets/urdf/franka_description/robots/franka_panda.urdf (robot description, URDF)
Before this commit: robot panda, 11 links, 10 joints
Links:
- added link panda_ee_finger
Joints:
- added joint panda_ee_finger: type fixed, parent panda_link7, child panda_ee_finger, origin xyz=0 0 0.207 rpy=0 0 0, axis 0 0 0

Commit message: Add ee link in urdf

File: assets/urdf/franka_description/robots/franka_panda.urdf (robot description, URDF)
Before this commit: robot panda, 11 links, 10 joints
Links:
- added link panda_ee
Joints:
- added joint panda_ee: type fixed, parent panda_link7, child panda_ee, origin xyz=0 0 0.23 rpy=0 0 0, axis 0 0 0

Commit message: Some improvements. But it tends to lose the cube on the way to move it. Also add collision cost to the table, split the finger controls, align the real and sim controls, use the grasp cost function, while loop for updating eta, fine tuning variance

File: assets/urdf/franka_description/robots/franka_panda.urdf (robot description, URDF)
Before this commit: robot panda, 12 links, 11 joints
Joints:
- joint panda_ee: origin xyz=0 0 0.23 rpy=0 0 0 -> xyz=0 0 0.21 rpy=0 0 0

Commit message: Video two success trials, but not use active inference

File: assets/urdf/franka_description/robots/franka_panda.urdf (robot description, URDF)
Before this commit: robot panda, 12 links, 11 joints
Joints:
- joint panda_ee: origin xyz=0 0 0.21 rpy=0 0 0 -> xyz=0 0 0.22 rpy=0 0 0
