Commit message: Added albert mppi, but urdf needs refinement because of werid behavior

File: assets/urdf/albert/albert.urdf (robot description, URDF)
Before this commit: robot albert, 26 links, 25 joints
Links:
- link rotacastor_left_link: mass 1 -> 0.01
- link rotacastor_right_link: mass 1 -> 0.01
- link wheel_left_link: mass 100 -> 1
- link wheel_right_link: mass 100 -> 1
Joints:
- joint rotacastor_left_joint: type continuous -> fixed
- joint rotacastor_right_joint: type continuous -> fixed

Commit message: adds albert. Set frictions to zero for rotacaster

File: assets/urdf/albert/albert.urdf (robot description, URDF)
Before this commit: robot albert, 26 links, 25 joints
Links:
- link chassis_link: mass 250 -> 150
- link internal_link: mass 31 -> 20
- link rotacastor_left_link: mass 0.01 -> 0.3
- link rotacastor_right_link: mass 0.01 -> 0.3
- link top_mount: mass 10 -> 8
- link top_mount_bottom: mass 10 -> 8
Joints:
- joint mmrobot_joint_top_mount: origin xyz=-0.15 0 0 rpy=0 0 0 -> xyz=0.237 0 0 rpy=0 0 0

Commit message: MOvements are better if I increase the mass of the  base and use only the navifation cost

File: assets/urdf/albert/albert.urdf (robot description, URDF)
Before this commit: robot albert, 26 links, 25 joints
Links:
- link chassis_link: mass 250 -> 2500
